File: Hardware/SensorNode/urban-climate-monitor.sch (KiCad schematic (older format))
At the start: 48 parts, among them J1 Conn_ARM_JTAG_SWD_10, U1 AAT1217, U2 TPS27081A, U3 SHT31-DIS, U4 24LC32, U5 TSD305, U6 ADG633YCP, U7 TSV911RILT, U8 RFM95W, U9 STM32L412KB

Commit message: Fix warnings of electrical rules check
Parts:
- U2: symbol my-symbols-library:TPS27081A -> my-symbols-library:TPS27081A_ForReversePolarityProtection
Connections:
- no-connect marks 14 -> 22
Other:
- moved on the sheet: FB1
Changed lines of the file:
@@
 $EndComp
 $Comp
-L my-symbols-library:TPS27081A U2
+L my-symbols-library:TPS27081A_ForReversePolarityProtection U2
 U 1 1 5F915AF3
 P 11300 2000
@@
 NoConn ~ 14450 2200
 Wire Wire Line
-	5700 8050 6150 8050
-Wire Wire Line
-	6800 7950 6800 8050
+	5900 8050 6350 8050
+Wire Wire Line
+	7500 7950 7500 8050
 $Comp
 L power:+3.3V #PWR036
 U 1 1 5FC51B03
-P 6800 7950
-F 0 "#PWR036" H 6800 7800 50  0001 C CNN
-F 1 "+3.3V" H 6815 8123 50  0000 C CNN
-F 2 "" H 6800 7950 50  0001 C CNN
-F 3 "" H 6800 7950 50  0001 C CNN
-	1    6800 7950
-	1    0    0    -1
-$EndComp
-Wire Wire Line
-	6350 8050 6800 8050
+P 7500 7950
+F 0 "#PWR036" H 7500 7800 50  0001 C CNN
+F 1 "+3.3V" H 7515 8123 50  0000 C CNN
+F 2 "" H 7500 7950 50  0001 C CNN
+F 3 "" H 7500 7950 50  0001 C CNN
+	1    7500 7950
+	1    0    0    -1
+$EndComp
+Wire Wire Line
+	7050 8050 7500 8050
 $Comp
 L Device:Ferrite_Bead_Small FB1
 U 1 1 5FC319BD
-P 6250 8050
-F 0 "FB1" V 6013 8050 50  0000 C CNN
-F 1 "Ferrite_Bead_Small" V 6104 8050 50  0000 C CNN
-F 2 "Inductor_SMD:L_0805_2012Metric_Pad1.05x1.20mm_HandSolder" V 6180 8050 50  0001 C CNN
-F 3 "~" H 6250 8050 50  0001 C CNN
-	1    6250 8050
+P 6950 8050
+F 0 "FB1" V 6713 8050 50  0000 C CNN
+F 1 "Ferrite_Bead_Small" V 6804 8050 50  0000 C CNN
+F 2 "Inductor_SMD:L_0805_2012Metric_Pad1.05x1.20mm_HandSolder" V 6880 8050 50  0001 C CNN
+F 3 "~" H 6950 8050 50  0001 C CNN
+	1    6950 8050
 	0    1    1    0
 $EndComp
@@
 Connection ~ 12400 4200
 Wire Wire Line
-	13200 4200 12400 4200
+	13200 4200 12800 4200
 Wire Wire Line
 	12400 4200 12400 4700
@@
 Text GLabel 4850 9250 0    50   Input ~ 0
 VIN_SENSE
-Connection ~ 5700 8050
-Wire Wire Line
-	5700 8050 5550 8050
+Connection ~ 5900 8050
+Wire Wire Line
+	5900 8050 5550 8050
 $Comp
 L power:+3.3VA #PWR035
 U 1 1 5FC71CDC
-P 5700 7950
-F 0 "#PWR035" H 5700 7800 50  0001 C CNN
-F 1 "+3.3VA" H 5715 8123 50  0000 C CNN
-F 2 "" H 5700 7950 50  0001 C CNN
-F 3 "" H 5700 7950 50  0001 C CNN
-	1    5700 7950
-	1    0    0    -1
-$EndComp
-Wire Wire Line
-	5700 7950 5700 8050
+P 5900 7950
+F 0 "#PWR035" H 5900 7800 50  0001 C CNN
+F 1 "+3.3VA" H 5915 8123 50  0000 C CNN
+F 2 "" H 5900 7950 50  0001 C CNN
+F 3 "" H 5900 7950 50  0001 C CNN
+	1    5900 7950
+	1    0    0    -1
+$EndComp
+Wire Wire Line
+	5900 7950 5900 8050
 $Comp
 L Device:C C2
@@
 Text Label 9650 4200 0    50   ~ 0
 PHOTO_VCC
+Wire Wire Line
+	5950 8350 6050 8350
+NoConn ~ 4850 9450
+NoConn ~ 4850 9550
+NoConn ~ 4850 9650
+NoConn ~ 6050 9850
+NoConn ~ 6050 9550
+NoConn ~ 6050 9450
+NoConn ~ 6050 9150
+NoConn ~ 6050 8350
+$Comp
+L power:PWR_FLAG #FLG0101
+U 1 1 5FAD5982
+P 12800 4050
+F 0 "#FLG0101" H 12800 4125 50  0001 C CNN
+F 1 "PWR_FLAG" H 12800 4223 50  0000 C CNN
+F 2 "" H 12800 4050 50  0001 C CNN
+F 3 "~" H 12800 4050 50  0001 C CNN
+	1    12800 4050
+	1    0    0    -1
+$EndComp
+Wire Wire Line
+	12800 4050 12800 4200
+Connection ~ 12800 4200
+Wire Wire Line
+	12800 4200 12400 4200
+$Comp
+L power:PWR_FLAG #FLG0102
+U 1 1 5FAFED66
+P 6350 7950
+F 0 "#FLG0102" H 6350 8025 50  0001 C CNN
+F 1 "PWR_FLAG" H 6350 8123 50  0000 C CNN
+F 2 "" H 6350 7950 50  0001 C CNN
+F 3 "~" H 6350 7950 50  0001 C CNN
+	1    6350 7950
+	1    0    0    -1
+$EndComp
+Wire Wire Line
+	6350 7950 6350 8050
+Connection ~ 6350 8050
+Wire Wire Line
+	6350 8050 6850 8050
+$Comp
+L power:PWR_FLAG #FLG?
+U 1 1 5FB294B7
+P 10000 1700
+F 0 "#FLG?" H 10000 1775 50  0001 C CNN
+F 1 "PWR_FLAG" H 10000 1873 50  0000 C CNN
+F 2 "" H 10000 1700 50  0001 C CNN
+F 3 "~" H 10000 1700 50  0001 C CNN
+	1    10000 1700
+	1    0    0    -1
+$EndComp
+Wire Wire Line
+	10000 1700 10000 1800
+Connection ~ 10000 1800
 $EndSCHEMATC

Commit message: Add photo enable pin, add deployment compose
Parts:
- R6: value 50k -> 10k
Changed lines of the file:
@@
 P 13500 4950
 F 0 "R6" H 13570 4996 50  0000 L CNN
-F 1 "50k" H 13570 4905 50  0000 L CNN
+F 1 "10k" H 13570 4905 50  0000 L CNN
 F 2 "Resistor_SMD:R_0805_2012Metric_Pad1.20x1.40mm_HandSolder" V 13430 4950 50  0001 C CNN
 F 3 "~" H 13500 4950 50  0001 C CNN
