File: hardware/sensor-node/sensor-node.sch (KiCad schematic (older format))
At the start: 46 parts, among them J1 Conn_ARM_JTAG_SWD_10, U1 AAT1217, U2 TPS27081A, U3 SHT31-DIS, U4 24LC32, U5 TSD305, U6 ADG633YCP, U7 TSV911RILT, U8 RFM95W, U9 STM32L412KB

Commit message: Update schema to include I2C voltage switching
Parts:
- removed U5: TSD305, Package_TO_SOT_THT:TO-5-4_Window, symbol my-symbols-library:TSD305
- added J?: Conn_Coaxial, symbol Connector:Conn_Coaxial
- added Q?: Q_PMOS_DGS, symbol Device:Q_PMOS_DGS
- added R?: 100k, Resistor_SMD:R_0805_2012Metric_Pad1.20x1.40mm_HandSolder, symbol Device:R
- added R? (x3): R, symbol Device:R
- added U5: MLX90614, Package_TO_SOT_THT:TO-39-4, symbol my-symbols-library:MLX90614
Connections:
- net labels added: I2C_ENABLE, VI2C
- wire segments 257 -> 279
- no-connect marks 22 -> 21
Other:
- note added: "5000nA Sleep"
- note added: "5000nA Standby"
- note added: "I2C Bus Control"
- note added: "I2C-Address: 0x5a"
- note removed: "10nA Standby"
- note removed: "20nA Sleep"
- note removed: "I2C-Address: 0x00"
- moved on the sheet: AE1, C10, H1, H2, R10, R11

Commit message: Update PCB, add debugging printouts to application
Parts:
- J1: renamed from J?; footprint (none) -> my-footprints-library:CONUFL001-SMD
- Q1: renamed from Q?; footprint (none) -> Package_TO_SOT_SMD:SOT-23; symbol Device:Q_PMOS_DGS -> Device:Q_PMOS_GSD
- U1, U2: footprint Package_TO_SOT_SMD:TSOT-23-6_HandSoldering -> Package_TO_SOT_SMD:TSOT-23-6
- Z1, Z2, Z3: renamed from R?; value R -> Z; footprint (none) -> Resistor_SMD:R_0805_2012Metric_Pad1.20x1.40mm_HandSolder
- gave numbers to parts that had none: 1
- renumbered C15 to C13, C13 to C14, C14 to C15, J1 to J2, R10 to R11, R11 to R12, R12 to R14
Connections:
- net +3V3: now also Q1.2 (S); no longer Q1.1 (D)
- net I2C_ENABLE: now also Q1.1 (G); no longer Q1.2 (G)
